File: template/Dax_Circuit/Dax_Circuit.kicad_sch (KiCad schematic)
At the start: 0 parts

Commit message: Update template
Other:
- title: (none) -> DAX-C00-@{if(("${VARIANT}"==""), "001", "${VARIANT}")}
Changed lines of the file:
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@@
 (kicad_sch
-	(version 20231120)
+	(version 20260306)
 	(generator "eeschema")
-	(generator_version "8.0")
+	(generator_version "10.0")
 	(paper "B")
 	(title_block
-		(rev "${REVISION}")
+		(title "DAX-C00-@{if((\"${VARIANT}\"==\"\"), \"001\", \"${VARIANT}\")}")
+		(rev "A1")
 	)
 	(image
@@
 		)
 	)
+	(embedded_fonts no)
 )
