File: template/Dax_Circuit/Dax_Circuit.kicad_sch (KiCad schematic)
At the start: 0 parts

Commit message: Add CIRCUIT_NUMBER variable
Other:
- title: DAX-C00-@{if(("${VARIANT}"==""), "001", "${VARIANT}")} -> DAX-C${CIRCUIT_NUMBER}-@{if(("${VARIANT}"==""), "001", "${VARIANT}")}
Changed lines of the file:
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@@
 	(paper "B")
 	(title_block
-		(title "DAX-C00-@{if((\"${VARIANT}\"==\"\"), \"001\", \"${VARIANT}\")}")
+		(title "DAX-C${CIRCUIT_NUMBER}-@{if((\"${VARIANT}\"==\"\"), \"001\", \"${VARIANT}\")}")
 		(rev "A1")
 	)
